File: Hardware/SparkFun_Soil_Moisture_Sensor.brd (EAGLE design)
At the start: 20.3 x 61 mm, 10 parts, among them Q1 2N3904

Commit message: V10
V10 prototype
Parts:
- removed U$1, U$2: (no value), SparkFun-Electromechanical:STAND-OFF
- added JP2: (no value), SparkFun-Connectors:SCREWTERMINAL-3.5MM-3
- added STANDOFF1, STANDOFF2: STAND-OFF, SparkFun-Electromechanical:STAND-OFF
- JP1: device SparkFun-Connectors:1X03 -> SparkFun-Connectors:MOLEX-1X3
- moved FRAME1 78.0 mm to (8.89, -10.2)
- moved LOGO1 61.9 mm to (33.0, 48.3)
- moved LOGO2 61.0 mm to (19.1, 47.0)
- moved U$4 59.1 mm to (22.9, 48.3)
- moved Q1 57.2 mm to (11.4, 49.5), turned to 0 degrees
- moved R1 57.2 mm to (14.0, 49.5), turned to 270 degrees
- moved R2 57.2 mm to (8.89, 49.5)
- moved JP1 56.0 mm to (8.89, 54.6), turned to 0 degrees
Connections:
- net GND: now also JP1.2, JP2.2; no longer JP1.1
- net SIG: now also JP1.3, JP2.1; no longer JP1.2
- net VCC: now also JP1.1, JP2.3; no longer JP1.3
Routing:
- net SIG: track 7.40 -> 12.3 mm
- net VCC: track 7.52 -> 10.0 mm
- net PROBE1: track 11.4 -> 12.6 mm
- net GND: track 8.83 -> 8.06 mm
- net PROBE2: track 10.9 -> 10.3 mm
Other:
- board size 20.3 x 61 mm -> 22.9 x 61 mm

Commit message: Soil moisture sensor v10 prototype
Soil moisture sensor v10 prototype
Parts:
- moved FRAME1 16.5 mm to (-7.62, -10.2)
- moved LOGO1 15.2 mm to (17.8, 48.3)
- moved U$4 5.24 mm to (17.8, 49.5)
Other:
- board text added: "How do I expose the probe pads?"
- board text added: "Joel Bartlett"
- board text added: "V10"
Changed lines of the file:
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@@
 <setting verticaltext="up"/>
 </settings>
-<grid distance="0.05" unitdist="inch" unit="inch" style="lines" multiple="1" display="yes" altdistance="0.001" altunitdist="inch" altunit="inch"/>
+<grid distance="0.05" unitdist="inch" unit="inch" style="lines" multiple="1" display="yes" altdistance="0.005" altunitdist="inch" altunit="inch"/>
 <layers>
 <layer number="1" name="Top" color="4" fill="1" visible="yes" active="yes"/>
@@
 <layer number="37" name="tTest" color="7" fill="1" visible="no" active="yes"/>
 <layer number="38" name="bTest" color="7" fill="1" visible="no" active="yes"/>
-<layer number="39" name="tKeepout" color="4" fill="11" visible="yes" active="yes"/>
+<layer number="39" name="tKeepout" color="4" fill="11" visible="no" active="yes"/>
 <layer number="40" name="bKeepout" color="1" fill="11" visible="no" active="yes"/>
 <layer number="41" name="tRestrict" color="4" fill="10" visible="no" active="yes"/>
@@
 <text x="15.9512" y="59.817" size="0.8128" layer="21" font="vector" ratio="15" rot="R180">SIG</text>
 <text x="9.0424" y="59.8424" size="0.8128" layer="21" font="vector" ratio="15" rot="R180">VCC</text>
-<text x="1.778" y="46.609" size="1.016" layer="21" font="vector" ratio="15">Soil Moisture Sensor</text>
-<text x="16.256" y="59.563" size="1.016" layer="22" font="vector" ratio="15" rot="SMR0">VCC</text>
-<text x="9.017" y="59.563" size="1.016" layer="22" font="vector" ratio="15" rot="SMR0">SIG</text>
+<text x="1.016" y="46.355" size="1.27" layer="21" font="vector" ratio="15">Soil Moisture Sensor</text>
+<text x="9.144" y="59.563" size="1.016" layer="22" font="vector" ratio="15" rot="SMR0">VCC</text>
+<text x="16.002" y="59.563" size="1.016" layer="22" font="vector" ratio="15" rot="SMR0">SIG</text>
 <text x="12.7" y="59.563" size="1.016" layer="22" font="vector" ratio="15" rot="SMR0">GND</text>
+<text x="19.05" y="-10.16" size="1.778" layer="51" font="vector" ratio="10">Joel Bartlett</text>
+<text x="13.208" y="46.101" size="1.27" layer="16" font="vector" ratio="15" rot="SMR0">V10</text>
+<dimension x1="7.62" y1="7.62" x2="15.24" y2="7.62" x3="11.43" y3="1.27" textsize="1.27" textratio="15" layer="51" unit="inch"/>
+<dimension x1="2.54" y1="58.42" x2="20.32" y2="58.42" x3="11.43" y3="62.23" textsize="1.27" textratio="15" layer="51" unit="inch"/>
+<text x="35.56" y="29.21" size="1.27" layer="51" font="vector" ratio="15">How do I expose the probe pads?</text>
 </plain>
 <attributes>
@@
 <attribute name="PROD_ID" value="RES-12438" x="8.89" y="49.53" size="1.778" layer="27" font="vector" ratio="15" rot="R90" display="off"/>
 </element>
-<element name="FRAME1" library="SparkFun-Aesthetics" package="CREATIVE_COMMONS" value="" x="8.89" y="-10.16">
-<attribute name="VERSION" value="v01" x="8.89" y="-10.16" size="1.778" layer="27" font="vector" ratio="15" display="off"/>
-<attribute name="DESIGNER" value="Joel Bartlett" x="8.89" y="-10.16" size="1.778" layer="27" font="vector" ratio="15" display="off"/>
+<element name="FRAME1" library="SparkFun-Aesthetics" package="CREATIVE_COMMONS" value="" x="-7.62" y="-10.16">
+<attribute name="VERSION" value="v01" x="-7.62" y="-10.16" size="1.778" layer="27" font="vector" ratio="15" display="off"/>
+<attribute name="DESIGNER" value="Joel Bartlett" x="-7.62" y="-10.16" size="1.778" layer="27" font="vector" ratio="15" display="off"/>
 </element>
-<element name="LOGO1" library="SparkFun-Aesthetics" package="SFE_LOGO_NAME_FLAME_.1" value="SFE_LOGO_NAME_FLAME.1_INCH" x="33.02" y="48.26" rot="MR0"/>
+<element name="LOGO1" library="SparkFun-Aesthetics" package="SFE_LOGO_NAME_FLAME_.1" value="SFE_LOGO_NAME_FLAME.1_INCH" x="17.78" y="48.26" rot="MR0"/>
 <element name="LOGO2" library="SparkFun-Aesthetics" package="OSHW-LOGO-S" value="OSHW-LOGOS" x="19.05" y="46.99" rot="MR0"/>
-<element name="U$4" library="SparkFun-Aesthetics" package="SFE_LOGO_FLAME_.2" value="" x="22.86" y="48.26"/>
+<element name="U$4" library="SparkFun-Aesthetics" package="SFE_LOGO_FLAME_.2" value="" x="17.78" y="49.53"/>
 <element name="JP1" library="SparkFun-Connectors" package="MOLEX-1X3" value="" x="8.89" y="54.61"/>
 <element name="JP2" library="SparkFun-Connectors" package="SCREWTERMINAL-3.5MM-3" value="" x="14.9098" y="57.3786" rot="R180"/>
@@
 <signal name="PROBE2">
 <contactref element="R2" pad="1"/>
-<polygon width="0.254" layer="1" isolate="0.3048">
+<polygon width="0.254" layer="1">
 <vertex x="0" y="44.45"/>
 <vertex x="0" y="0"/>
@@
 <wire x1="3.81" y1="48.26" x2="3.81" y2="43.18" width="0.254" layer="1"/>
 <via x="3.81" y="43.18" extent="1-16" drill="0.508"/>
-<polygon width="0.254" layer="16" isolate="0.3048">
+<polygon width="0.254" layer="16">
 <vertex x="0" y="44.45"/>
 <vertex x="0" y="0"/>
