File: Hardware/SparkFun_Soil_Moisture_Sensor.sch (EAGLE design)
At the start: 7 parts, among them Q1 2N3904

Commit message: V10
V10 prototype
Parts:
- added JP2: (no value), SparkFun-Connectors:M03SCREW
- added STANDOFF1, STANDOFF2: STAND-OFF, SparkFun-Electromechanical:STAND-OFF
- FRAME1: DESIGNER (none) -> Joel Bartlett
- JP1: device SparkFun-Connectors:M03PTH -> SparkFun-Connectors:M03POLAR
Connections:
- net GND: now also JP1.2, JP2.2; no longer JP1.1
- net SIG: now also JP1.3, JP2.1; no longer JP1.2
- net VCC: now also JP1.1, JP2.3; no longer JP1.3
Other:
- note added: "Based off the Soil Moisture Circuit found at: http://www.faludi.com/2006/11/02/moisture-sensor-circuit/"
- note added: "Connectors:"
- note added: "Probe Circuit"
- note added: "Rod length and spacing were not the most significant variables. In general you want the probes long enough to reach the moist soil and not so close together that they are likely to touch accidentally. Keeping them about an inch apart works great. The big variable is the composition of the soil itselfj (especially salts), so ideally you would calibrate for each type of soil. -Rob Faludi"
- note added: "Test different values for R1 to get lower power consumption while still getting a good ADC reading."
- note removed: "Test different values for R1 to get better power consumption while still getting a good ADC reading."
- moved on the sheet: JP1, Q1, R1, R2

Commit message: Soil moisture sensor v10 prototype
Soil moisture sensor v10 prototype
Other:
- note added: "Connectors: JST Jumper 3 Wire Assembly - PRT-09915 Screw Terminals 3.5mm Pitch (3-Pin) - PRT-08235"
- note added: "Rod length and spacing were not the most significant variables. In general you want the probes long enough to reach the moist soil and not so close together that they are likely to touch accidentally. Keeping them about an inch apart works great. The big variable is the composition of the soil itself (especially salts), so ideally you would calibrate for each type of soil. -Rob Faludi"
- note removed: "Connectors:"
- note removed: "Rod length and spacing were not the most significant variables. In general you want the probes long enough to reach the moist soil and not so close together that they are likely to touch accidentally. Keeping them about an inch apart works great. The big variable is the composition of the soil itselfj (especially salts), so ideally you would calibrate for each type of soil. -Rob Faludi"
Changed lines of the file:
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@@
 In general you want the probes long enough to reach the moist soil and not so close together that they are likely to touch accidentally.
 Keeping them about an inch apart works great.
-The big variable is the composition of the soil itselfj (especially salts), so ideally you would calibrate for each type of soil.
+The big variable is the composition of the soil itself (especially salts), so ideally you would calibrate for each type of soil.
 -Rob Faludi</text>
-<text x="45.72" y="170.18" size="1.778" layer="95">Connectors: </text>
+<text x="30.48" y="165.1" size="1.778" layer="95">Connectors:
+JST Jumper 3 Wire Assembly - PRT-09915
+Screw Terminals 3.5mm Pitch (3-Pin) - PRT-08235</text>
 <text x="167.64" y="172.72" size="1.778" layer="95">Probe Circuit</text>
 </plain>
